File: board-ring-magnet/magnet-motor-encoder-as5304.sch (KiCad schematic (older format))
At the start: 6 parts, among them U1 DS18B20, U2 AS5304

Commit message: board as5304: add AO and GND test points
Parts:
- added W1: GND, symbol TEST_1P
- added W2: AO, symbol TEST_1P
Connections:
- wire segments 30 -> 32
Changed lines of the file:
@@
 $EndComp
 $Comp
-L GND #PWR5
+L GND #PWR6
 U 1 1 5781651B
 P 5100 3450
-F 0 "#PWR5" H 5100 3200 50  0001 C CNN
+F 0 "#PWR6" H 5100 3200 50  0001 C CNN
 F 1 "GND" H 5100 3300 50  0000 C CNN
 F 2 "" H 5100 3450 50  0000 C CNN
@@
 	5350 3450 5100 3450
 $Comp
-L GND #PWR8
+L GND #PWR9
 U 1 1 57816542
 P 6800 3450
-F 0 "#PWR8" H 6800 3200 50  0001 C CNN
+F 0 "#PWR9" H 6800 3200 50  0001 C CNN
 F 1 "GND" H 6800 3300 50  0000 C CNN
 F 2 "" H 6800 3450 50  0000 C CNN
@@
 	6350 3450 6800 3450
 $Comp
-L +5V #PWR9
+L +5V #PWR10
 U 1 1 5781658C
 P 6800 3850
-F 0 "#PWR9" H 6800 3700 50  0001 C CNN
+F 0 "#PWR10" H 6800 3700 50  0001 C CNN
 F 1 "+5V" H 6800 3990 50  0000 C CNN
 F 2 "" H 6800 3850 50  0000 C CNN
@@
 $EndComp
 $Comp
-L +5V #PWR6
+L +5V #PWR7
 U 1 1 578165A6
 P 5100 3650
-F 0 "#PWR6" H 5100 3500 50  0001 C CNN
+F 0 "#PWR7" H 5100 3500 50  0001 C CNN
 F 1 "+5V" H 5100 3790 50  0000 C CNN
 F 2 "" H 5100 3650 50  0000 C CNN
@@
 $EndComp
 $Comp
-L +5V #PWR7
+L +5V #PWR8
 U 1 1 578165BC
 P 5100 4050
-F 0 "#PWR7" H 5100 3900 50  0001 C CNN
+F 0 "#PWR8" H 5100 3900 50  0001 C CNN
 F 1 "+5V" H 5100 4190 50  0000 C CNN
 F 2 "" H 5100 4050 50  0000 C CNN
@@
 	5100 4050 5350 4050
 $Comp
-L GND #PWR10
+L GND #PWR11
 U 1 1 578165DD
 P 6800 3950
-F 0 "#PWR10" H 6800 3700 50  0001 C CNN
+F 0 "#PWR11" H 6800 3700 50  0001 C CNN
 F 1 "GND" H 6800 3800 50  0000 C CNN
 F 2 "" H 6800 3950 50  0000 C CNN
@@
 $EndComp
 $Comp
-L +5V #PWR11
+L +5V #PWR12
 U 1 1 57816CAD
 P 7700 3550
-F 0 "#PWR11" H 7700 3400 50  0001 C CNN
+F 0 "#PWR12" H 7700 3400 50  0001 C CNN
 F 1 "+5V" H 7700 3690 50  0000 C CNN
 F 2 "" H 7700 3550 50  0000 C CNN
@@
 	7850 4000 7850 3950
 $Comp
-L GND #PWR12
+L GND #PWR13
 U 1 1 57816CFE
 P 7700 4050
-F 0 "#PWR12" H 7700 3800 50  0001 C CNN
+F 0 "#PWR13" H 7700 3800 50  0001 C CNN
 F 1 "GND" H 7700 3900 50  0000 C CNN
 F 2 "" H 7700 4050 50  0000 C CNN
@@
 Wire Wire Line
 	5100 4150 5350 4150
+$Comp
+L TEST_1P W2
+U 1 1 578189A0
+P 5000 3950
+F 0 "W2" H 5000 4220 50  0000 C CNN
+F 1 "AO" H 5000 4150 50  0000 C CNN
+F 2 "" H 5200 3950 50  0000 C CNN
+F 3 "" H 5200 3950 50  0000 C CNN
+	1    5000 3950
+	0    -1   -1   0
+$EndComp
+Wire Wire Line
+	5000 3950 5350 3950
+$Comp
+L TEST_1P W1
+U 1 1 57818B75
+P 7100 4800
+F 0 "W1" H 7100 5070 50  0000 C CNN
+F 1 "GND" H 7100 5000 50  0000 C CNN
+F 2 "" H 7300 4800 50  0000 C CNN
+F 3 "" H 7300 4800 50  0000 C CNN
+	1    7100 4800
+	1    0    0    -1
+$EndComp
+$Comp
+L GND #PWR5
+U 1 1 57818CC1
+P 7100 5000
+F 0 "#PWR5" H 7100 4750 50  0001 C CNN
+F 1 "GND" H 7100 4850 50  0000 C CNN
+F 2 "" H 7100 5000 50  0000 C CNN
+F 3 "" H 7100 5000 50  0000 C CNN
+	1    7100 5000
+	1    0    0    -1
+$EndComp
+Wire Wire Line
+	7100 4800 7100 5000
 $EndSCHEMATC

Commit message: board AS5304: add Power LED
Parts:
- added D?: PWR, symbol LED
- added R?: 1k, symbol R
Connections:
- wire segments 32 -> 35
Changed lines of the file:
@@
 P 6800 3850
 F 0 "#PWR10" H 6800 3700 50  0001 C CNN
-F 1 "+5V" H 6800 3990 50  0000 C CNN
+F 1 "+5V" V 6800 4050 50  0000 C CNN
 F 2 "" H 6800 3850 50  0000 C CNN
 F 3 "" H 6800 3850 50  0000 C CNN
@@
 P 6800 3950
 F 0 "#PWR11" H 6800 3700 50  0001 C CNN
-F 1 "GND" H 6800 3800 50  0000 C CNN
+F 1 "GND" V 6800 3750 50  0000 C CNN
 F 2 "" H 6800 3950 50  0000 C CNN
 F 3 "" H 6800 3950 50  0000 C CNN
@@
 Wire Wire Line
 	7100 4800 7100 5000
+$Comp
+L +5V #PWR?
+U 1 1 57823139
+P 8600 3550
+F 0 "#PWR?" H 8600 3400 50  0001 C CNN
+F 1 "+5V" H 8600 3690 50  0000 C CNN
+F 2 "" H 8600 3550 50  0000 C CNN
+F 3 "" H 8600 3550 50  0000 C CNN
+	1    8600 3550
+	1    0    0    -1
+$EndComp
+$Comp
+L GND #PWR?
+U 1 1 5782315C
+P 8600 4650
+F 0 "#PWR?" H 8600 4400 50  0001 C CNN
+F 1 "GND" H 8600 4500 50  0000 C CNN
+F 2 "" H 8600 4650 50  0000 C CNN
+F 3 "" H 8600 4650 50  0000 C CNN
+	1    8600 4650
+	1    0    0    -1
+$EndComp
+$Comp
+L LED D?
+U 1 1 578231AB
+P 8600 3900
+F 0 "D?" H 8600 4000 50  0000 C CNN
+F 1 "PWR" H 8600 3800 50  0000 C CNN
+F 2 "" H 8600 3900 50  0000 C CNN
+F 3 "" H 8600 3900 50  0000 C CNN
+	1    8600 3900
+	0    -1   -1   0
+$EndComp
+$Comp
+L R R?
+U 1 1 57823260
+P 8600 4350
+F 0 "R?" V 8680 4350 50  0000 C CNN
+F 1 "1k" V 8600 4350 50  0000 C CNN
+F 2 "" V 8530 4350 50  0000 C CNN
+F 3 "" H 8600 4350 50  0000 C CNN
+	1    8600 4350
+	1    0    0    -1
+$EndComp
+Wire Wire Line
+	8600 3550 8600 3700
+Wire Wire Line
+	8600 4100 8600 4200
+Wire Wire Line
+	8600 4500 8600 4650
 $EndSCHEMATC

Commit message: board as5304: modified solder jumper; ERC passed
Parts:
- gave numbers to parts that had none: 2
Changed lines of the file:
@@
 $EndComp
 $Comp
-L GND #PWR6
+L GND #PWR01
 U 1 1 5781651B
 P 5100 3450
-F 0 "#PWR6" H 5100 3200 50  0001 C CNN
+F 0 "#PWR01" H 5100 3200 50  0001 C CNN
 F 1 "GND" H 5100 3300 50  0000 C CNN
 F 2 "" H 5100 3450 50  0000 C CNN
@@
 	5350 3450 5100 3450
 $Comp
-L GND #PWR9
+L GND #PWR02
 U 1 1 57816542
 P 6800 3450
-F 0 "#PWR9" H 6800 3200 50  0001 C CNN
+F 0 "#PWR02" H 6800 3200 50  0001 C CNN
 F 1 "GND" H 6800 3300 50  0000 C CNN
 F 2 "" H 6800 3450 50  0000 C CNN
@@
 	6350 3450 6800 3450
 $Comp
-L +5V #PWR10
+L +5V #PWR03
 U 1 1 5781658C
 P 6800 3850
-F 0 "#PWR10" H 6800 3700 50  0001 C CNN
+F 0 "#PWR03" H 6800 3700 50  0001 C CNN
 F 1 "+5V" V 6800 4050 50  0000 C CNN
 F 2 "" H 6800 3850 50  0000 C CNN
@@
 $EndComp
 $Comp
-L +5V #PWR7
+L +5V #PWR04
 U 1 1 578165A6
 P 5100 3650
-F 0 "#PWR7" H 5100 3500 50  0001 C CNN
+F 0 "#PWR04" H 5100 3500 50  0001 C CNN
 F 1 "+5V" H 5100 3790 50  0000 C CNN
 F 2 "" H 5100 3650 50  0000 C CNN
@@
 $EndComp
 $Comp
-L +5V #PWR8
+L +5V #PWR05
 U 1 1 578165BC
 P 5100 4050
-F 0 "#PWR8" H 5100 3900 50  0001 C CNN
+F 0 "#PWR05" H 5100 3900 50  0001 C CNN
 F 1 "+5V" H 5100 4190 50  0000 C CNN
 F 2 "" H 5100 4050 50  0000 C CNN
@@
 	5100 4050 5350 4050
 $Comp
-L GND #PWR11
+L GND #PWR06
 U 1 1 578165DD
 P 6800 3950
-F 0 "#PWR11" H 6800 3700 50  0001 C CNN
+F 0 "#PWR06" H 6800 3700 50  0001 C CNN
 F 1 "GND" V 6800 3750 50  0000 C CNN
 F 2 "" H 6800 3950 50  0000 C CNN
@@
 $EndComp
 $Comp
-L +5V #PWR12
+L +5V #PWR07
 U 1 1 57816CAD
 P 7700 3550
-F 0 "#PWR12" H 7700 3400 50  0001 C CNN
+F 0 "#PWR07" H 7700 3400 50  0001 C CNN
 F 1 "+5V" H 7700 3690 50  0000 C CNN
 F 2 "" H 7700 3550 50  0000 C CNN
@@
 	7850 4000 7850 3950
 $Comp
-L GND #PWR13
+L GND #PWR08
 U 1 1 57816CFE
 P 7700 4050
-F 0 "#PWR13" H 7700 3800 50  0001 C CNN
+F 0 "#PWR08" H 7700 3800 50  0001 C CNN
 F 1 "GND" H 7700 3900 50  0000 C CNN
 F 2 "" H 7700 4050 50  0000 C CNN
@@
 $EndComp
 $Comp
-L GND #PWR3
+L GND #PWR09
 U 1 1 5781721E
 P 2950 4850
-F 0 "#PWR3" H 2950 4600 50  0001 C CNN
+F 0 "#PWR09" H 2950 4600 50  0001 C CNN
 F 1 "GND" H 2950 4700 50  0000 C CNN
 F 2 "" H 2950 4850 50  0000 C CNN
@@
 	2750 4850 2950 4850
 $Comp
-L +5V #PWR4
+L +5V #PWR010
 U 1 1 5781790E
 P 2950 5050
-F 0 "#PWR4" H 2950 4900 50  0001 C CNN
+F 0 "#PWR010" H 2950 4900 50  0001 C CNN
 F 1 "+5V" H 2950 5190 50  0000 C CNN
 F 2 "" H 2950 5050 50  0000 C CNN
@@
 $EndComp
 $Comp
-L GND #PWR2
+L GND #PWR011
 U 1 1 57817C4A
 P 2650 4050
-F 0 "#PWR2" H 2650 3800 50  0001 C CNN
+F 0 "#PWR011" H 2650 3800 50  0001 C CNN
 F 1 "GND" H 2650 3900 50  0000 C CNN
 F 2 "" H 2650 4050 50  0000 C CNN
@@
 $EndComp
 $Comp
-L +5V #PWR1
+L +5V #PWR012
 U 1 1 57817C64
 P 2650 3750
-F 0 "#PWR1" H 2650 3600 50  0001 C CNN
+F 0 "#PWR012" H 2650 3600 50  0001 C CNN
 F 1 "+5V" H 2650 3890 50  0000 C CNN
 F 2 "" H 2650 3750 50  0000 C CNN
@@
 $EndComp
 $Comp
-L GND #PWR5
+L GND #PWR013
 U 1 1 57818CC1
 P 7100 5000
-F 0 "#PWR5" H 7100 4750 50  0001 C CNN
+F 0 "#PWR013" H 7100 4750 50  0001 C CNN
 F 1 "GND" H 7100 4850 50  0000 C CNN
 F 2 "" H 7100 5000 50  0000 C CNN
@@
 	7100 4800 7100 5000
 $Comp
-L +5V #PWR?
+L +5V #PWR014
 U 1 1 57823139
 P 8600 3550
-F 0 "#PWR?" H 8600 3400 50  0001 C CNN
+F 0 "#PWR014" H 8600 3400 50  0001 C CNN
 F 1 "+5V" H 8600 3690 50  0000 C CNN
 F 2 "" H 8600 3550 50  0000 C CNN
@@
 $EndComp
 $Comp
-L GND #PWR?
+L GND #PWR015
 U 1 1 5782315C
 P 8600 4650
-F 0 "#PWR?" H 8600 4400 50  0001 C CNN
+F 0 "#PWR015" H 8600 4400 50  0001 C CNN
 F 1 "GND" H 8600 4500 50  0000 C CNN
 F 2 "" H 8600 4650 50  0000 C CNN
@@
 $EndComp
 $Comp
-L LED D?
+L LED D1
 U 1 1 578231AB
 P 8600 3900
-F 0 "D?" H 8600 4000 50  0000 C CNN
+F 0 "D1" H 8600 4000 50  0000 C CNN
 F 1 "PWR" H 8600 3800 50  0000 C CNN
 F 2 "" H 8600 3900 50  0000 C CNN
@@
 $EndComp
 $Comp
-L R R?
+L R R1
 U 1 1 57823260
 P 8600 4350
-F 0 "R?" V 8680 4350 50  0000 C CNN
+F 0 "R1" V 8680 4350 50  0000 C CNN
 F 1 "1k" V 8600 4350 50  0000 C CNN
 F 2 "" V 8530 4350 50  0000 C CNN

Commit message: board as5304: footprints selected, netlist created
Parts:
- C1, C2: footprint (none) -> Capacitors_SMD:C_0805
- D1: footprint (none) -> LEDs:LED_0805
- JP1: footprint (none) -> Pin_Headers:Pin_Header_Straight_1x05
- R1: footprint (none) -> Resistors_SMD:R_0805
- SJ1: footprint (none) -> open-project:S_JUMPER_3
- U1: footprint (none) -> TO_SOT_Packages_THT:TO-92_Inline_Narrow_Oval
- U2: footprint (none) -> Housings_SSOP:TSSOP-20_4.4x6.5mm_Pitch0.65mm
- W1, W2: footprint (none) -> SMD_Packages:1Pin
Changed lines of the file:
@@
 F 0 "U2" H 5850 4500 60  0000 C CNN
 F 1 "AS5304" H 5850 3300 60  0000 C CNN
-F 2 "" H 5850 3900 60  0000 C CNN
+F 2 "Housings_SSOP:TSSOP-20_4.4x6.5mm_Pitch0.65mm" H 5850 3900 60  0001 C CNN
 F 3 "" H 5850 3900 60  0000 C CNN
 	1    5850 3900
@@
 F 0 "C1" H 7575 3900 50  0000 L CNN
 F 1 "100n" H 7575 3700 50  0000 L CNN
-F 2 "" H 7588 3650 50  0000 C CNN
+F 2 "Capacitors_SMD:C_0805" H 7588 3650 50  0001 C CNN
 F 3 "" H 7550 3800 50  0000 C CNN
 	1    7550 3800
@@
 F 0 "C2" H 7875 3900 50  0000 L CNN
 F 1 "10µ" H 7875 3700 50  0000 L CNN
-F 2 "" H 7888 3650 50  0000 C CNN
+F 2 "Capacitors_SMD:C_0805" H 7888 3650 50  0001 C CNN
 F 3 "" H 7850 3800 50  0000 C CNN
 	1    7850 3800
@@
 F 0 "U1" H 2300 5200 50  0000 C CNN
 F 1 "DS18B20" H 2450 4700 50  0000 C CNN
-F 2 "" H 2300 5200 50  0000 C CNN
+F 2 "TO_SOT_Packages_THT:TO-92_Inline_Narrow_Oval" H 2300 5200 50  0001 C CNN
 F 3 "" H 2300 5200 50  0000 C CNN
 	1    2450 4950
@@
 F 0 "JP1" H 3300 4200 60  0000 C CNN
 F 1 "RCA_ENCODER_PSK" H 3300 3600 60  0000 C CNN
-F 2 "" H 3300 3900 60  0000 C CNN
+F 2 "Pin_Headers:Pin_Header_Straight_1x05" H 3300 3900 60  0001 C CNN
 F 3 "" H 3300 3900 60  0000 C CNN
 	1    3300 3900
@@
 F 0 "SJ1" H 4150 5150 60  0000 C CNN
 F 1 "TMP / IDX" H 4400 4800 60  0000 C CNN
-F 2 "" H 4400 4550 60  0000 C CNN
+F 2 "open-project:S_JUMPER_3" H 4400 4550 60  0001 C CNN
 F 3 "" H 4400 4550 60  0000 C CNN
 	1    4400 4950
@@
 F 0 "W2" H 5000 4220 50  0000 C CNN
 F 1 "AO" H 5000 4150 50  0000 C CNN
-F 2 "" H 5200 3950 50  0000 C CNN
+F 2 "SMD_Packages:1Pin" H 5200 3950 50  0001 C CNN
 F 3 "" H 5200 3950 50  0000 C CNN
 	1    5000 3950
@@
 F 0 "W1" H 7100 5070 50  0000 C CNN
 F 1 "GND" H 7100 5000 50  0000 C CNN
-F 2 "" H 7300 4800 50  0000 C CNN
+F 2 "SMD_Packages:1Pin" H 7300 4800 50  0001 C CNN
 F 3 "" H 7300 4800 50  0000 C CNN
 	1    7100 4800
@@
 F 0 "D1" H 8600 4000 50  0000 C CNN
 F 1 "PWR" H 8600 3800 50  0000 C CNN
-F 2 "" H 8600 3900 50  0000 C CNN
+F 2 "LEDs:LED_0805" H 8600 3900 50  0001 C CNN
 F 3 "" H 8600 3900 50  0000 C CNN
 	1    8600 3900
@@
 F 0 "R1" V 8680 4350 50  0000 C CNN
 F 1 "1k" V 8600 4350 50  0000 C CNN
-F 2 "" V 8530 4350 50  0000 C CNN
+F 2 "Resistors_SMD:R_0805" V 8530 4350 50  0001 C CNN
 F 3 "" H 8600 4350 50  0000 C CNN
 	1    8600 4350

Commit message: board as5304: add test point library; replace measurement point footprint
Parts:
- W1, W2: footprint SMD_Packages:1Pin -> Measurement_Points:Measurement_Point_Round-SMD-Pad_Small
Changed lines of the file:
@@
 F 0 "W2" H 5000 4220 50  0000 C CNN
 F 1 "AO" H 5000 4150 50  0000 C CNN
-F 2 "SMD_Packages:1Pin" H 5200 3950 50  0001 C CNN
+F 2 "Measurement_Points:Measurement_Point_Round-SMD-Pad_Small" H 5200 3950 50  0001 C CNN
 F 3 "" H 5200 3950 50  0000 C CNN
 	1    5000 3950
@@
 F 0 "W1" H 7100 5070 50  0000 C CNN
 F 1 "GND" H 7100 5000 50  0000 C CNN
-F 2 "SMD_Packages:1Pin" H 7300 4800 50  0001 C CNN
+F 2 "Measurement_Points:Measurement_Point_Round-SMD-Pad_Small" H 7300 4800 50  0001 C CNN
 F 3 "" H 7300 4800 50  0000 C CNN
 	1    7100 4800

Commit message: board as5304: named signals in schematic
Connections:
- net labels added: A, AO, B, IDX, TMP, TMP_IDX
Changed lines of the file:
@@
 Wire Wire Line
 	8600 4500 8600 4650
+Text Label 4400 4350 0    60   ~ 0
+TMP_IDX
+Text Label 5100 4950 0    60   ~ 0
+IDX
+Text Label 3550 4950 0    60   ~ 0
+TMP
+Text Label 3950 3950 0    60   ~ 0
+A
+Text Label 3950 4050 0    60   ~ 0
+B
+Text Label 5100 3950 0    60   ~ 0
+AO
 $EndSCHEMATC

Commit message: board as5304: fix component values
Parts:
- JP1: value RCA_ENCODER_PSK -> ENCODER
- SJ1: value TMP / IDX -> TMP/IDX
- U2: value AS5304 -> AS5304(A)
Changed lines of the file:
@@
 P 5850 3900
 F 0 "U2" H 5850 4500 60  0000 C CNN
-F 1 "AS5304" H 5850 3300 60  0000 C CNN
+F 1 "AS5304(A)" H 5850 3300 60  0000 C CNN
 F 2 "Housings_SSOP:TSSOP-20_4.4x6.5mm_Pitch0.65mm" H 5850 3900 60  0001 C CNN
 F 3 "" H 5850 3900 60  0000 C CNN
@@
 P 3300 3900
 F 0 "JP1" H 3300 4200 60  0000 C CNN
-F 1 "RCA_ENCODER_PSK" H 3300 3600 60  0000 C CNN
+F 1 "ENCODER" H 3300 3600 60  0000 C CNN
 F 2 "Pin_Headers:Pin_Header_Straight_1x05" H 3300 3900 60  0001 C CNN
 F 3 "" H 3300 3900 60  0000 C CNN
@@
 P 4400 4950
 F 0 "SJ1" H 4150 5150 60  0000 C CNN
-F 1 "TMP / IDX" H 4400 4800 60  0000 C CNN
+F 1 "TMP/IDX" H 4400 4800 60  0000 C CNN
 F 2 "open-project:S_JUMPER_3" H 4400 4550 60  0001 C CNN
 F 3 "" H 4400 4550 60  0000 C CNN
