File: board-as5045b/magnet-motor-encoder_v1.sch (EAGLE design)
At the start: 14 parts, among them IC1 AS5045B, IC3 DS18B20

Commit message: board as5045b: new board shape (imported from 3d-model/solidworks); rev4 tag
Parts:
- C1: device resistor:C-EUC0805K -> rcl:R-EU_R0603
Other:
- moved on the sheet: C1
Changed lines of the file:
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@@
 <part name="R2" library="resistor" deviceset="R-EU_" device="R0805" value="1k"/>
 <part name="R3" library="resistor" deviceset="R-EU_" device="R0805" value="1k"/>
-<part name="C1" library="resistor" deviceset="C-EU" device="C0805K" value="100n"/>
+<part name="C1" library="rcl" deviceset="R-EU_" device="R0603" value="100n"/>
 <part name="C2" library="resistor" deviceset="C-EU" device="C0805K" value="10µ"/>
 <part name="SJ1" library="rca_sontiges" deviceset="SJ" device="S" value="3V3?"/>
@@
 <wire x1="-129.54" y1="-40.64" x2="-119.38" y2="-40.64" width="0.1524" layer="91"/>
 <wire x1="-119.38" y1="-40.64" x2="-111.76" y2="-40.64" width="0.1524" layer="91"/>
-<wire x1="-119.38" y1="-43.18" x2="-119.38" y2="-40.64" width="0.1524" layer="91"/>
+<wire x1="-124.46" y1="-48.26" x2="-119.38" y2="-40.64" width="0.1524" layer="91"/>
 <junction x="-119.38" y="-40.64"/>
 <pinref part="C3" gate="G$1" pin="2"/>
@@
 <wire x1="-106.68" y1="-55.88" x2="-119.38" y2="-55.88" width="0.1524" layer="91"/>
 <pinref part="C1" gate="G$1" pin="1"/>
-<wire x1="-119.38" y1="-55.88" x2="-119.38" y2="-50.8" width="0.1524" layer="91"/>
+<wire x1="-119.38" y1="-55.88" x2="-114.3" y2="-48.26" width="0.1524" layer="91"/>
 <wire x1="-106.68" y1="-55.88" x2="-91.44" y2="-55.88" width="0.1524" layer="91"/>
 <pinref part="C2" gate="G$1" pin="1"/>

Commit message: board as5045b: add missing CSn pulldown resistor; new rev5 tag
Parts:
- added R4: 4k7, resistor:R-EU_R0805
Connections:
- new net N$4: IC1.CSN, R4.2
- net GND: now also R4.1
Changed lines of the file:
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@@
 <part name="GND6" library="rca_sontiges" deviceset="GND" device=""/>
 <part name="P+7" library="supply1" deviceset="+5V" device=""/>
+<part name="GND7" library="rca_sontiges" deviceset="GND" device=""/>
+<part name="R4" library="resistor" deviceset="R-EU_" device="R0805" value="4k7"/>
 </parts>
 <sheets>
@@
 <instance part="GND6" gate="1" x="-22.86" y="-60.96"/>
 <instance part="P+7" gate="1" x="-22.86" y="-35.56"/>
+<instance part="GND7" gate="1" x="38.1" y="-27.94"/>
+<instance part="R4" gate="G$1" x="38.1" y="-15.24" rot="R90"/>
 </instances>
 <busses>
@@
 <wire x1="-22.86" y1="-58.42" x2="-22.86" y2="-55.88" width="0.1524" layer="91"/>
 </segment>
+<segment>
+<pinref part="GND7" gate="1" pin="GND"/>
+<pinref part="R4" gate="G$1" pin="1"/>
+<wire x1="38.1" y1="-25.4" x2="38.1" y2="-20.32" width="0.1524" layer="91"/>
+</segment>
 </net>
 <net name="A" class="0">
@@
 </segment>
 </net>
+<net name="N$4" class="0">
+<segment>
+<pinref part="IC1" gate="G$1" pin="CSN"/>
+<pinref part="R4" gate="G$1" pin="2"/>
+<wire x1="17.78" y1="-5.08" x2="38.1" y2="-5.08" width="0.1524" layer="91"/>
+<wire x1="38.1" y1="-5.08" x2="38.1" y2="-10.16" width="0.1524" layer="91"/>
+</segment>
+</net>
